File: CATSTNC-R2.kicad_pcb (KiCad board)
At the start: 2 copper layers, 79 x 59.5 mm, 50 parts, among them J1 Conn_Coaxial, J4 USB_C_Receptacle_USB2.0, J5 DC IN, J6 GPIO-1, J7 GPIO-2, SW1 RESET, SW2 RESET, U1 NCP1117-5.0_SOT223, U2 W25Q128JVS, U3 RP2040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

Commit message: Improve design
Parts:
- removed C1: 0.1uF, Capacitor_THT:C_Disc_D3.4mm_W2.1mm_P2.50mm
- added C15: 100nF, Capacitor_SMD:C_0402_1005Metric, F.Cu at (121.4, 107.4)
- added C17: 100nF, Capacitor_SMD:C_0402_1005Metric, F.Cu at (129.0, 99.0)
- added C18: 1uF, Capacitor_SMD:C_0402_1005Metric, F.Cu at (121.0, 97.7)
- added C19: 100nF, Capacitor_SMD:C_0402_1005Metric, F.Cu at (132.7, 102.5)
- added C20: 100nF, Capacitor_SMD:C_0402_1005Metric, F.Cu at (118.0, 102.4)
- C11, C12, C14, C6, C7, C8, C9: footprint Capacitor_SMD:C_0805_2012Metric -> Capacitor_SMD:C_0402_1005Metric
- C3: footprint Capacitor_THT:CP_Radial_D5.0mm_P2.50mm -> Capacitor_SMD:C_0805_2012Metric
- R3, R4, R5, R6, R7, R8: footprint Resistor_SMD:R_0805_2012Metric -> Resistor_SMD:R_0402_1005Metric
- SW2: value RESET -> BOOT
- moved R7 23.1 mm to (123.8, 93.2), turned to 45 degrees
- moved R8 21.7 mm to (123.0, 92.4), turned to 45 degrees
- moved C12 17.8 mm to (133.4, 103.2), turned to 45 degrees
- moved C3 16.7 mm to (176.0, 119.3), turned to 0 degrees
- moved R3 5.61 mm to (116.7, 88.2), turned to -45 degrees
- moved C8 2.70 mm to (120.8, 92.1)
- moved R5 2.60 mm to (134.3, 72.3), turned to 180 degrees
- moved R6 2.60 mm to (138.9, 72.3), turned to 180 degrees
- moved C9 1.63 mm to (124.6, 94.3)
- moved C14 1.50 mm to (126.6, 96.1), turned to 135 degrees
- moved R4 0.87 mm to (131.8, 105.9)
- moved C7 0.84 mm to (133.3, 107.4)
- moved G*** 0.82 mm to (153.7, 89.3)
- moved C11 0.73 mm to (118.0, 103.4)
- moved SW2 0.60 mm to (111.1, 85.5), turned to 0 degrees
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Connections:
- J4 pad A6: Net-(J4-D+-PadA6) -> D+
- J4 pad A7: Net-(J4-D--PadA7) -> D-
- J4 pad B6: Net-(J4-D+-PadA6) -> D+
- J4 pad B7: Net-(J4-D--PadA7) -> D-
- R7 pad 1: Net-(J4-D--PadA7) -> Net-(U3-USB_DM)
- R8 pad 1: Net-(J4-D+-PadA6) -> Net-(U3-USB_DP)
- U3 pad 2: UART_TX -> unconnected-(U3-GPIO0-Pad2)
- U3 pad 3: UART_RX -> unconnected-(U3-GPIO1-Pad3)
- U3 pad 46: D- -> Net-(U3-USB_DM)
- U3 pad 47: D+ -> Net-(U3-USB_DP)
Routing:
- net +3V3: track 143.6 -> 172.3 mm, vias 4 -> 3
- net +5V: track 151.9 -> 138.0 mm, vias 0 -> 1
- net GND: track 71.2 -> 80.8 mm, vias 12 -> 19
- net +1V1: track 23.2 -> 31.8 mm, vias 2 -> 3
- net Net-(U3-USB_DP): track 0.00 -> 7.00 mm
- net Net-(J4-D+-PadA6): track 6.62 -> 0.00 mm
- net Net-(U3-USB_DM): track 0.00 -> 6.15 mm
- net Net-(J4-D--PadA7): track 5.63 -> 0.00 mm
- net Net-(J4-CC1): track 4.95 -> 2.50 mm
- net Net-(J4-CC2): track 4.18 -> 2.11 mm
- net Net-(C7-Pad1): track 3.86 -> 2.84 mm
- net D+: track 29.4 -> 30.4 mm
- net SDN: track 41.5 -> 40.8 mm
- net IRQ: track 37.0 -> 36.3 mm
- net XOUT: track 5.26 -> 4.62 mm
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Other:
- board text added: "PWR"
- board text added: "RX"
- board text added: "TX"
- board text added: "USB"

Commit message: Rev 2 Ordered
Parts:
- removed U1: NCP1117-5.0_SOT223, Package_TO_SOT_SMD:SOT-223-3_TabPin2
- added U5: LM7805_TO220, Package_TO_SOT_THT:TO-220-3_Vertical, F.Cu at (110.1, 88.8)
- C2, C5: value 8.2pF -> 7.5pF; footprint Capacitor_THT:C_Disc_D3.4mm_W2.1mm_P2.50mm -> Capacitor_SMD:C_0402_1005Metric
- C4: value 12pF -> 13pF; footprint Capacitor_THT:C_Disc_D3.4mm_W2.1mm_P2.50mm -> Capacitor_SMD:C_0402_1005Metric
- L1, L2: value 25nH -> 24nH; footprint Inductor_THT:L_Toroid_Horizontal_D6.5mm_P10.00mm_Diameter7-5mm_Amidon-T25 -> Inductor_SMD:L_0402_1005Metric
- R7, R8: value 27 -> 27 or 22
- moved SW1 33.0 mm to (124.6, 83.9)
- moved C16 17.9 mm to (111.4, 76.5), turned to -90 degrees
- moved C10 17.7 mm to (129.5, 75.4)
- moved C4 11.4 mm to (170.6, 87.4), turned to 180 degrees
- moved U4 9.34 mm to (133.4, 82.8), turned to -90 degrees
- moved L2 8.87 mm to (171.1, 84.0), turned to 90 degrees
- moved SW2 7.38 mm to (118.3, 83.9), turned to 180 degrees
- moved C5 5.45 mm to (170.6, 80.6), turned to 180 degrees
- moved C2 4.44 mm to (170.6, 94.2), turned to 180 degrees
- moved L1 1.84 mm to (171.1, 90.8), turned to 90 degrees
- moved C13 1.25 mm to (111.4, 73.0)
Connections:
- net VBUS renamed VCC
- C2 pad 2: GND -> GNDA
- C4 pad 2: GND -> GNDA
- C5 pad 2: GND -> GNDA
- J1 pad 2: GND -> GNDA
- U6 pad 15: GND -> GNDA
Routing:
- net GND: track 80.8 -> 18.7 mm, vias 19 -> 21
- net GNDA: track 0.00 -> 40.9 mm
- net VCC: track 29.0 -> 43.7 mm, vias 0 -> 1
- net +3V3: track 172.3 -> 163.1 mm, vias 3 -> 1
- net Net-(U3-RUN): track 21.7 -> 28.3 mm
- net Net-(C4-Pad1): track 12.4 -> 5.83 mm
- net Net-(J1-In): track 14.5 -> 9.19 mm
- net +5V: track 138.0 -> 142.7 mm
- net Net-(U6-ANT): track 8.63 -> 6.94 mm
- net SDN: track 40.8 -> 42.3 mm
- net IRQ: track 36.3 -> 37.9 mm
- net Net-(R3-Pad1): track 4.11 -> 5.04 mm
Other:
- board text added: "JLCJLCJLCJLC"

Commit message: Start work on Rev 3
Parts:
- removed C13: 100uF, Capacitor_THT:CP_Radial_D5.0mm_P2.50mm
- removed U5: LM7805_TO220, Package_TO_SOT_THT:TO-220-3_Vertical
- added C1: 100nF, Capacitor_SMD:C_0603_1608Metric, F.Cu at (109.0, 77.2)
- added C21: 22uF, Capacitor_SMD:C_0603_1608Metric, F.Cu at (116.5, 82.5)
- added C22: 22uF, Capacitor_SMD:C_0603_1608Metric, F.Cu at (116.5, 84.1)
- added C23: 100nF, Capacitor_SMD:C_0603_1608Metric, F.Cu at (116.5, 85.7)
- added C24: 100nF, Capacitor_SMD:C_0603_1608Metric, F.Cu at (109.0, 73.7)
- added C25: 10uF, Capacitor_SMD:C_0805_2012Metric, F.Cu at (111.0, 73.7)
- added C26: 10uF, Capacitor_SMD:C_0805_2012Metric, F.Cu at (113.2, 73.7)
- added C27: 33nF, Capacitor_SMD:C_0603_1608Metric, F.Cu at (113.5, 77.2)
- added D1: BAT54C, Package_TO_SOT_SMD:SOT-23, F.Cu at (120.1, 80.5)
- added L3: 6.8uH, Inductor_SMD:L_Sunlord_SWPA6020S, F.Cu at (111.5, 84.1)
- added R1: 54.9K 1%, Resistor_SMD:R_0402_1005Metric, F.Cu at (115.7, 80.5)
- added R13: 0, Resistor_SMD:R_0603_1608Metric, F.Cu at (111.3, 79.7)
- added R2: 10.0K 1%, Resistor_SMD:R_0402_1005Metric, F.Cu at (115.7, 78.5)
- added U1: TPS62933, Package_TO_SOT_SMD:SOT-583-8, F.Cu at (111.2, 77.2)
- C10, C16: footprint Capacitor_THT:CP_Radial_D5.0mm_P2.50mm -> Capacitor_SMD:C_1206_3216Metric
- J1: value Conn_Coaxial -> BNC
- moved SW2 18.9 mm to (137.0, 81.5)
- moved C16 16.7 mm to (128.0, 75.0), turned to 90 degrees
- moved SW1 12.4 mm to (137.0, 85.0)
- moved U4 7.65 mm to (125.8, 83.7)
- moved C10 1.08 mm to (130.5, 75.0)
Connections:
- net XIN renamed Net-(U3-XIN)
- net XOUT renamed Net-(U3-XOUT)
- C16 pad 1: +5V -> VCC
- J4 pad A4: unconnected-(J4-VBUS-PadA4) -> USB_VBUS
- J4 pad A9: unconnected-(J4-VBUS-PadA4) -> USB_VBUS
- J4 pad B4: unconnected-(J4-VBUS-PadA4) -> USB_VBUS
- J4 pad B9: unconnected-(J4-VBUS-PadA4) -> USB_VBUS
- U4 pad 3: VCC -> +5V
Routing:
- net +3V3: track 163.1 -> 71.6 mm, vias 1 -> 0
- net +5V: track 142.7 -> 68.5 mm
- net VCC: track 43.7 -> 0.00 mm, vias 1 -> 0
- net Net-(U3-RUN): track 28.3 -> 2.36 mm, vias 2 -> 1
- net D-: track 30.4 -> 5.36 mm, vias 2 -> 0
- net D+: track 30.5 -> 6.33 mm, vias 2 -> 0
- net RT: track 0.00 -> 7.17 mm, vias 0 -> 2
- net unconnected-(J4-VBUS-PadA4): track 6.93 -> 0.00 mm
- net Net-(R3-Pad1): track 5.04 -> 0.00 mm
- net Net-(U1-SS): track 0.00 -> 2.94 mm
- net GND: vias 21 -> 17
Other:
- board text added: "CATS Base Transceiver Rev. 3 Designed by Cam Kerby VE3KCN Oct. 2024"
- board text removed: "CATS Base Transceiver Rev. 2 Designed by Cam Kerby VE3KCN Nov. 2023"

Commit message: More work on Rev 3
Parts:
- turned SW1 to 180 degrees
Routing:
- net +3V3: track 71.6 -> 163.5 mm, vias 0 -> 5
- net +5V: track 68.5 -> 128.6 mm, vias 1 -> 3
- net USB_VBUS: track 0.00 -> 31.2 mm, vias 0 -> 2
- net D-: track 5.36 -> 31.8 mm
- net D+: track 6.33 -> 32.1 mm
- net VCC: track 0.00 -> 21.7 mm
- net Net-(R3-Pad1): track 0.00 -> 21.5 mm, vias 0 -> 2
- net Net-(U3-RUN): track 2.36 -> 23.6 mm, vias 1 -> 2
- net REG_5V: track 0.00 -> 10.1 mm
- net Net-(U1-SW): track 0.00 -> 7.74 mm
- net VFB: track 0.00 -> 5.56 mm
- net Net-(U1-BST): track 0.00 -> 2.89 mm
- net GND: track 18.7 -> 19.7 mm
Other:
- board text added: "CATS Base Transceiver Rev. 3 Designed by Cam Kerby VE3KCN Sept. 2024"
- board text removed: "CATS Base Transceiver Rev. 3 Designed by Cam Kerby VE3KCN Oct. 2024"
