File: CATSTNC-R2.kicad_pcb (KiCad board)
At the start: 2 copper layers, 79 x 59.5 mm, 66 parts, among them J1 BNC, J4 USB_C_Receptacle_USB2.0, J5 DC IN, J6 GPIO-1, J7 GPIO-2, SW1 RESET, SW2 BOOT, U1 TPS62933, U2 W25Q128JVS, U3 RP2040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

Commit message: Add power mux, USB TVS
Parts:
- removed D1: BAT54C, Package_TO_SOT_SMD:SOT-23
- added C13: 10uF, Capacitor_SMD:C_0402_1005Metric, F.Cu at (116.8, 79.6)
- added C28: 10uF, Capacitor_SMD:C_0402_1005Metric, F.Cu at (121.4, 82.7)
- added C29: 10uF, Capacitor_SMD:C_0402_1005Metric, F.Cu at (121.4, 80.7)
- added C30: 10uF, Capacitor_SMD:C_0402_1005Metric, F.Cu at (118.3, 79.2)
- added R17: 54.9K 1%, Resistor_SMD:R_0402_1005Metric, F.Cu at (117.6, 81.6)
- added R18: 15.0K 1%, Resistor_SMD:R_0402_1005Metric, F.Cu at (117.6, 83.6)
- added R19: 10K, Resistor_SMD:R_0402_1005Metric, F.Cu at (120.8, 79.2)
- added U5: TPS2116DRL, Package_TO_SOT_SMD:SOT-583-8, F.Cu at (119.5, 81.2)
- added U7: USBLC6-2SC6, Package_TO_SOT_SMD:SOT-23-6, F.Cu at (136.7, 75.0)
- C21, C22, C23: footprint Capacitor_SMD:C_0603_1608Metric -> Capacitor_SMD:C_0402_1005Metric
- moved C23 1.62 mm to (116.0, 84.2)
- moved R3 1.47 mm to (117.7, 89.2), turned to 135 degrees
- moved C22 1.12 mm to (116.0, 83.1)
- moved U4 1.10 mm to (126.5, 84.5)
- moved C21 0.68 mm to (116.0, 82.1)
Connections:
- J4 pad A6: D+ -> Net-(J4-D+-PadA6)
- J4 pad A7: D- -> Net-(J4-D--PadA7)
- J4 pad B6: D+ -> Net-(J4-D+-PadA6)
- J4 pad B7: D- -> Net-(J4-D--PadA7)
- U3 pad 4: unconnected-(U3-GPIO2-Pad4) -> MUX_ST
Routing:
- net MUX_ST: track 0.00 -> 35.6 mm, vias 0 -> 2
- net USB_VBUS: track 31.2 -> 42.5 mm, vias 2 -> 3
- net +5V: track 128.6 -> 137.7 mm
- net D+: track 32.0 -> 23.8 mm
- net Net-(J4-D+-PadA6): track 0.00 -> 6.64 mm
- net D-: track 31.9 -> 25.3 mm
- net Net-(J4-D--PadA7): track 0.00 -> 5.84 mm
- net GND: track 19.7 -> 24.9 mm, vias 17 -> 25
- net +3V3: track 163.5 -> 167.5 mm, vias 5 -> 4
- net Net-(U5-PR1): track 0.00 -> 2.22 mm
- net REG_5V: track 10.1 -> 11.5 mm
- net QSPI_SS: track 23.7 -> 24.2 mm
